File: v3.0-Dev-Kit/v3.0-Dev-Kit.kicad_pcb (KiCad board)
At the start: 2 copper layers, 42 x 59 mm, 33 parts, among them J1 8 Pin Header, SW1 Up, SW2 Down, SW3 Left, SW4 Right, SW5 botton, U1 WeMos D1 Mini

Commit message: update colliding trace
Parts:
- removed the G*** at (0.00, 0.00) (x19)
- added G*** (x19): LOGO, LOGO, F.Cu at (0.00, 0.00)
Routing:
- net Net-(Brd1-Pad2): track 82.3 -> 100.8 mm, vias 1 -> 2

Commit message: export BOM and positioning files
Parts:
- removed the G*** at (0.00, 0.00) (x19)
- added G*** (x19): LOGO, LOGO, F.Cu at (0.00, 0.00)
Changed lines of the file:
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@@
   )
   (setup
-    (last_trace_width 0.4)
+    (last_trace_width 0.25)
     (user_trace_width 0.35)
     (user_trace_width 0.4)
